Commit message: Invert upper mast direction

File: urdf/knighttime_description.urdf (robot description, URDF)
Before this commit: robot knighttime_description_node, 6 links, 5 joints
Joints:
- joint second_stage_joint: axis 0 1 0 -> 0 -1 0

Commit message: Add effort limits

File: urdf/knighttime_description.urdf (robot description, URDF)
Before this commit: robot knighttime_description_node, 6 links, 5 joints
Joints:
- joint extension_joint: limit lower=0 upper=0.3048 effort=0 velocity=0 -> lower=0 upper=0.3048 effort=1 velocity=0
- joint main_mast_joint: limit lower=-1.57 upper=1.57 effort=0 velocity=2.856 -> lower=-1.57 upper=1.57 effort=1 velocity=2.856
- joint second_stage_joint: limit lower=-2.70526 upper=2.70526 effort=0 velocity=3.06796 -> lower=-2.70526 upper=2.70526 effort=1 velocity=3.06796
